File: PCB/Radiant.kicad_sch (KiCad schematic)
At the start: 19 parts, among them J1 Conn_01x04, SW1 RotaryEncoder_Switch, SW5 SW_Push, SW6 SW_Push, SW7 SW_Push, SW8 SW_Push, U1 XIAO-ESP32-C3-DIP

Commit message: Updated RadiantOS
Parts:
- J1: value Conn_01x04 -> Display 128*64
Connections:
- net GND: now also D1.2 (VSS), D2.2 (VSS), D3.2 (VSS), D4.2 (VSS), D5.2 (VSS), D6.2 (VSS), D7.2 (VSS)
- net VOUT+: now reaches D1.4 (VDD), D2.4 (VDD), D3.4 (VDD), D4.4 (VDD), D5.4 (VDD), D6.4 (VDD), D7.4 (VDD)
- net 5V+: no longer names the net of U1.14 (VBUS)
Changed lines of the file:
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@@
+	(wire
+		(pts
+			(xy 63.5 60.96) (xy 81.28 60.96)
+		)
+		(stroke
+			(width 0)
+			(type default)
+		)
+	)
 	(wire
 		(pts
@@
 	(wire
 		(pts
-			(xy 63.5 60.96) (xy 81.28 60.96)
-		)
-		(stroke
-			(width 0)
-			(type default)
-		)
-	)
-	(wire
-		(pts
 			(xy 71.12 36.83) (xy 92.71 36.83)
 		)
@@
 		)
 	)
+	(global_label "GND"
+		(shape input)
+		(at 237.49 52.07 270)
+		(fields_autoplaced yes)
+		(effects
+			(font
+				(size 1.27 1.27)
+			)
+			(justify right)
+		)
+		(property "Intersheetrefs" "${INTERSHEET_REFS}"
+			(at 237.49 58.9257 90)
+			(effects
+				(font
+					(size 1.27 1.27)
+				)
+				(justify right)
+				(hide yes)
+			)
+		)
+	)
 	(global_label "s1 ec"
 		(shape input)
@@
 		)
 	)
-	(global_label "5V+"
-		(shape input)
-		(at 119.38 60.96 0)
+	(global_label "VOUT+"
+		(shape input)
+		(at 237.49 36.83 90)
 		(fields_autoplaced yes)
 		(effects
@@
 		)
 		(property "Intersheetrefs" "${INTERSHEET_REFS}"
-			(at 126.2357 60.96 0)
+			(at 237.49 27.5552 90)
 			(effects
 				(font
@@
 			)
 		)
-		(property "Value" "Conn_01x04"
+		(property "Value" "Display 128*64"
 			(at 218.44 87.6299 0)
 			(effects
